File: hardware/tug/tug.kicad_pcb (KiCad board)
At the start: 2 copper layers, 99.1 x 66.3 mm, 52 parts, among them J1 Conn_01x04, J2 Conn_01x04, J3 Conn_01x03, J4 Conn_01x03, J5 Conn_01x03, J6 Conn_01x02, J7 Conn_01x02, J8 Conn_01x02, P1 Digital, P10 CONN_01X01, P11 CONN_01X01, P12 CONN_01X01, P13 CONN_01X01, P2 Power, P3 Analog, P4 Analog, P5 PWM, P6 PWM, P7 Communication, P8 CONN_01X01, P9 CONN_01X01, Q1 Q_NMOS_GDS, Q2 Q_NMOS_GDS, Q3 Q_NMOS_GDS, Q4 Q_NMOS_GDS, U1 MC33883, U2 MLX91210

Commit message: Added v2 PCB
Parts:
- added J10: Conn_01x01, Pin_Headers:Pin_Header_Straight_1x01_Pitch2.54mm, F.Cu at (149.1, 66.0)
- added J11: Conn_01x01, Pin_Headers:Pin_Header_Straight_1x01_Pitch2.54mm, F.Cu at (108.7, 70.6)
- added J9: Conn_01x01, Pin_Headers:Pin_Header_Straight_1x01_Pitch2.54mm, F.Cu at (166.4, 123.7)
- added R14: 3.5mR, Resistors_SMD:R_2512, F.Cu at (115.1, 106.7)
- J3, J4, J5: value Conn_01x03 -> Conn_01x02; footprint Pin_Headers:Pin_Header_Straight_1x03_Pitch2.54mm -> Pin_Headers:Pin_Header_Straight_1x02_Pitch2.54mm
- U2: value MLX91210 -> INA240
- moved U2 3.98 mm to (114.0, 113.5), turned to 270 degrees
- moved C8 3.31 mm to (112.0, 120.1)
- moved C7 1.61 mm to (112.0, 117.9), turned to 180 degrees
Connections:
- C8 pad 1: /A0 -> +5V
- U2 pad 1: /SRC_HS1 -> /M1
- U2 pad 2: /SRC_HS1 -> GND
- U2 pad 3: /M1 -> GND
- U2 pad 4: /M1 -> GND
- U2 pad 5: GND -> /A0
- U2 pad 6: GND -> +5V
- U2 pad 7: /A0 -> +5V
- U2 pad 8: +5V -> /SRC_HS1
Routing:
- net /M1: track 0.00 -> 9.84 mm
- net /SRC_HS1: track 44.1 -> 53.7 mm
- net /A0: track 52.6 -> 43.9 mm
- net GND: track 476.2 -> 470.8 mm
- net +5V: track 160.3 -> 165.3 mm
- net /M2: vias 5 -> 4
Other:
- rule pad_to_mask_clearance: 0 -> 0.1016
- board text added: "Tug v2"
- board text removed: "Tug v1"

Commit message: WIP
Parts:
- moved R14 1.37 mm to (115.6, 108.0)
Routing:
- net /SRC_HS1: track 53.7 -> 50.8 mm
- net /M1: track 9.84 -> 8.01 mm
Changed lines of the file:
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@@
   )
   (setup
-    (last_trace_width 1.27)
+    (last_trace_width 0.635)
     (user_trace_width 0.254)
     (user_trace_width 0.381)
@@
       (padsonsilk false)
       (subtractmaskfromsilk false)
-      (outputformat 1)
+      (outputformat 4)
       (mirror false)
       (drillshape 0)
       (scaleselection 1)
-      (outputdirectory fab/v2/))
+      (outputdirectory doc/))
   )
   (net 0 "")
@@
   )
   (module Resistors_SMD:R_2512 (layer F.Cu)
-    (at 115.062 106.68 180)
+    (at 115.57 107.95 180)
     (descr "Resistor SMD 2512, reflow soldering, Vishay (see dcrcw.pdf)")
     (tags "resistor 2512")
@@
   (segment (start 158.677 113.792) (end 154.305 109.42) (width 3.81) (layer F.Cu) (net 94))
   (via (at 161.036 113.792) (size 3.048) (drill 2.032) (layers F.Cu B.Cu) (net 94))
-  (segment (start 113.919 111.633) (end 110.871 111.633) (width 0.635) (layer F.Cu) (net 95))
-  (segment (start 114.046 111.506) (end 113.919 111.633) (width 0.635) (layer F.Cu) (net 95))
-  (segment (start 114.046 107.188) (end 114.046 111.506) (width 0.635) (layer F.Cu) (net 95))
-  (segment (start 111.962 106.68) (end 113.538 106.68) (width 0.635) (layer F.Cu) (net 95))
-  (segment (start 113.538 106.68) (end 114.046 107.188) (width 0.635) (layer F.Cu) (net 95))
+  (segment (start 113.605 107.95) (end 114.3 108.645) (width 0.635) (layer F.Cu) (net 95))
+  (segment (start 112.47 107.95) (end 113.605 107.95) (width 0.635) (layer F.Cu) (net 95))
+  (segment (start 114.3 108.645) (end 114.3 110.744) (width 0.635) (layer F.Cu) (net 95))
+  (segment (start 113.411 111.633) (end 110.871 111.633) (width 0.635) (layer F.Cu) (net 95))
+  (segment (start 114.3 110.744) (end 113.411 111.633) (width 0.635) (layer F.Cu) (net 95))
   (segment (start 144.145 96.835) (end 144.145 100.27) (width 0.635) (layer F.Cu) (net 96))
   (segment (start 130.81 100.27) (end 130.81 98.52) (width 0.635) (layer F.Cu) (net 97))
@@
   (segment (start 135.254999 89.534999) (end 135.254999 99.186999) (width 0.635) (layer F.Cu) (net 106))
   (segment (start 116.9035 111.633) (end 117.221 111.633) (width 0.635) (layer F.Cu) (net 106))
-  (segment (start 115.443 111.633) (end 117.221 111.633) (width 0.635) (layer F.Cu) (net 106))
-  (segment (start 115.316 111.506) (end 115.443 111.633) (width 0.635) (layer F.Cu) (net 106))
-  (segment (start 118.162 106.68) (end 115.824 106.68) (width 0.635) (layer F.Cu) (net 106))
-  (segment (start 115.316 107.188) (end 115.316 111.506) (width 0.635) (layer F.Cu) (net 106))
-  (segment (start 115.824 106.68) (end 115.316 107.188) (width 0.635) (layer F.Cu) (net 106))
+  (segment (start 116.459 111.633) (end 117.221 111.633) (width 0.635) (layer F.Cu) (net 106))
+  (segment (start 116.078 111.252) (end 116.459 111.633) (width 0.635) (layer F.Cu) (net 106))
+  (segment (start 116.078 109.407) (end 116.078 111.252) (width 0.635) (layer F.Cu) (net 106))
+  (segment (start 118.67 107.95) (end 117.535 107.95) (width 0.635) (layer F.Cu) (net 106))
+  (segment (start 117.535 107.95) (end 116.078 109.407) (width 0.635) (layer F.Cu) (net 106))
   (zone (net 95) (net_name /M1) (layer F.Cu) (hatch edge 0.508)
     (connect_pads yes (clearance 0.3048))
@@
     (polygon
       (pts
-        (xy 106.934 102.362) (xy 106.934 108.458) (xy 112.522 108.458) (xy 112.522 104.902) (xy 110.236 104.902)
+        (xy 106.934 102.362) (xy 106.934 109.728) (xy 113.03 109.728) (xy 113.03 106.172) (xy 110.236 106.172)
         (xy 110.236 103.886) (xy 110.236 102.362)
       )
@@
     (polygon
       (pts
-        (xy 117.348 109.474) (xy 117.348 104.902) (xy 128.524 104.902) (xy 131.318 104.902) (xy 134.366 98.044)
+        (xy 117.856 109.474) (xy 117.856 104.902) (xy 128.524 104.902) (xy 131.318 104.902) (xy 134.366 98.044)
         (xy 139.7 98.044) (xy 139.7 102.616) (xy 135.89 102.616) (xy 135.382 103.378) (xy 134.112 106.172)
         (xy 134.112 114.3) (xy 122.682 114.3) (xy 121.666 113.284) (xy 117.602 109.474)
