File: hardware/tug/tug.sch (KiCad schematic (older format))
At the start: 52 parts, among them J1 Conn_01x04, J2 Conn_01x04, J3 Conn_01x03, J4 Conn_01x03, J5 Conn_01x03, J6 Conn_01x02, J7 Conn_01x02, J8 Conn_01x02, P1 Digital, P10 CONN_01X01, P11 CONN_01X01, P12 CONN_01X01, P13 CONN_01X01, P2 Power, P3 Analog, P4 Analog, P5 PWM, P6 PWM, P7 Communication, P8 CONN_01X01, P9 CONN_01X01, Q1 Q_NMOS_GDS, Q2 Q_NMOS_GDS, Q3 Q_NMOS_GDS, Q4 Q_NMOS_GDS, U1 MC33883, U2 MLX91210

Commit message: Added v2 PCB
Parts:
- removed J3, J4, J5: Conn_01x03, Pin_Headers:Pin_Header_Straight_1x03_Pitch2.54mm, symbol conn:Conn_01x03
- removed U2: MLX91210, SMD_Packages:SOIC-8-N, symbol mlx91210:MLX91210
- added J10, J11, J9: Conn_01x01, Pin_Headers:Pin_Header_Straight_1x01_Pitch2.54mm, symbol conn:Conn_01x01
- added J3, J4, J5: Conn_01x02, Pin_Headers:Pin_Header_Straight_1x02_Pitch2.54mm, symbol conn:Conn_01x02
- added R14: 3.5mR, Resistors_SMD:R_2512, symbol device:R
- added U2: INA240, SMD_Packages:SOIC-8-N, symbol ina240:INA240
Connections:
- wire segments 213 -> 219
Other:
- note added: "Full range = 0.0035 * 13 * 50 = 2.275\nPower dissipation = 0.0017 * 13 * 13 = 0.5915W"
- note added: "Gain = 50 (INA240A2)"

Commit message: Switched current sensor to INA240
Other:
- note added: "Full range = 0.0035 * 13 * 50 = 2.275\nPower dissipation = 0.0035 * 13 * 13 = 0.5915W"
- note removed: "Full range = 0.0035 * 13 * 50 = 2.275\nPower dissipation = 0.0017 * 13 * 13 = 0.5915W"
Changed lines of the file:
@@
 EESchema Schematic File Version 4
-LIBS:tug-cache
 EELAYER 26 0
 EELAYER END
@@
 Sheet 1 1
 Title ""
-Date "mar. 31 mars 2015"
+Date "2018-07-03"
 Rev ""
 Comp ""
@@
 Gain = 50 (INA240A2)
 Text Notes 5450 4300 0    50   ~ 0
-Full range = 0.0035 * 13 * 50 = 2.275\nPower dissipation = 0.0017 * 13 * 13 = 0.5915W
+Full range = 0.0035 * 13 * 50 = 2.275\nPower dissipation = 0.0035 * 13 * 13 = 0.5915W
 $Comp
 L conn:Conn_01x01 J10
